File: sample1/sample.sch (KiCad schematic (older format))
At the start: 9 parts, among them M1 text_F_SilkS, M2 title=%T date=%D rev=%R comp=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, M3 %AsyPN, M4 text_F_Cu, M5 Assembly %AsyPN, Rev %AsyRev, M6 %T %PCBPN, M7 %F.Cu:%PCBPN - %PCBRev, M8 text_auto_date, M9 UserTitleBlock

Commit message: Update to KiCad v5 and make into Action Script.
Parts:
- M1: symbol text_F_SilkS -> autotext:text_F_SilkS
- M2, M5, M7: symbol text_auto -> autotext:text_auto
- M3: symbol BarcodeCode39 -> autotext:BarcodeCode39
- M4: symbol text_F_Cu -> autotext:text_F_Cu
- M6: symbol BarcodeCode128 -> autotext:BarcodeCode128
- M8: symbol text_auto_date -> autotext:text_auto_date
- M9: symbol UserTitleBlock -> autotext:UserTitleBlock
Other:
- note added: "Code 39 and Code 128 Barcodes"
- note added: "Formatted text fields"
- note added: "Put whatever fields and layout you like here\nonly rule is that the component must \nbe called "UserTitleBlock""
- note added: "Simple text fields"
- note added: "The following substitutions are performed:\n\nStandard keys:\n %F the file base name\n %DT today's date\n \nThe following are read from the title block of the corresponding schematic file:\n %T Project title\n %R Revision\n %D Issue Date\n %Y Company\n %C0 Comment 1\n %C1 Comment 2\n %C2 Comment 3\n %C3 Comment 4\n \nAdditional substitutions are made according to user defined \nfields from compon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"
- note added: "The same substitutions as for formatted text fields are performed.\n"
- note added: "Value field is replaced \nby today's date\n"
